File: daughter-board/stm32l476/stm32l476.kicad_pcb (KiCad board)
At the start: 2 copper layers, 33 x 91.4 mm, 49 parts, among them J1 Conn_02x10_Odd_Even, J2 Conn_02x10_Odd_Even, U1 STM32L476RG, Y1 Crystal_Small

Commit message: Uddate board design
Connections:
- J1 pad 6: unconnected-(J1-Pin_6-Pad6) -> /D4_MCU_PC1
- U1 pad 16: /D9_MCU_RX -> unconnected-(U1-PA2-Pad16)
- U1 pad 17: /D10_MCU_TX -> unconnected-(U1-PA3-Pad17)
- U1 pad 9: unconnected-(U1-PC1-Pad9) -> /D4_MCU_PC1
Routing:
- net /D9_MCU_RX: track 52.7 -> 0.00 mm
- net /D4_MCU_PC1: track 0.00 -> 51.9 mm
- net /D10_MCU_TX: track 30.0 -> 0.00 mm
