File: daughter-board/stm32l476/stm32l476.kicad_sch (KiCad schematic)
At the start: 49 parts, among them J1 Conn_02x10_Odd_Even, J2 Conn_02x10_Odd_Even, U1 STM32L476RG, Y1 Crystal_Small

Commit message: Uddate board design
Connections:
- net D10_MCU_TX: no longer U1.17 (PA3)
- net D9_MCU_RX: no longer U1.16 (PA2)
- net D4_MCU_PC1: now reaches U1.9 (PC1)
- net D4_MCU_PC1: now also J1.6 (Pin_6)
- no-connect marks 117 -> 115
Other:
- note removed: "UART2"
Changed lines of the file:
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@@
   (no_connect (at 248.92 96.52))
   (no_connect (at 200.66 96.52))
-  (no_connect (at 54.61 102.87))
   (no_connect (at 59.69 34.29))
   (no_connect (at 165.1 91.44))
@@
   (no_connect (at 165.1 81.28))
   (no_connect (at 248.92 91.44))
-  (no_connect (at 165.1 88.9))
   (no_connect (at 200.66 73.66))
   (no_connect (at 248.92 71.12))
@@
     (stroke (width 0) (type default))
   )
-  (wire (pts (xy 200.66 50.8) (xy 205.74 50.8))
-    (stroke (width 0) (type default))
-  )
   (wire (pts (xy 139.7 86.36) (xy 139.7 88.9))
     (stroke (width 0) (type default))
@@
     (stroke (width 0) (type default))
   )
-  (wire (pts (xy 205.74 57.15) (xy 205.74 50.8))
+  (wire (pts (xy 54.61 80.01) (xy 54.61 102.87))
     (stroke (width 0) (type default))
   )
@@
     (stroke (width 0) (type default))
   )
-  (wire (pts (xy 200.66 48.26) (xy 208.28 48.26))
-    (stroke (width 0) (type default))
-  )
   (wire (pts (xy 187.96 38.1) (xy 187.96 35.56))
     (stroke (width 0) (type default))
@@
     (stroke (width 0) (type default))
   )
-  (wire (pts (xy 208.28 54.61) (xy 222.25 54.61))
-    (stroke (width 0) (type default))
-  )
   (wire (pts (xy 52.07 115.57) (xy 52.07 130.81))
     (stroke (width 0) (type default))
@@
     (stroke (width 0) (type default))
   )
+  (wire (pts (xy 149.86 88.9) (xy 165.1 88.9))
+    (stroke (width 0) (type default))
+  )
   (wire (pts (xy 180.34 35.56) (xy 180.34 33.02))
     (stroke (width 0) (type default))
@@
     (stroke (width 0) (type default))
   )
-  (wire (pts (xy 208.28 48.26) (xy 208.28 54.61))
-    (stroke (width 0) (type default))
-  )
   (wire (pts (xy 182.88 132.08) (xy 182.88 129.54))
     (stroke (width 0) (type default))
@@
     (stroke (width 0) (type default))
   )
-  (wire (pts (xy 205.74 57.15) (xy 222.25 57.15))
-    (stroke (width 0) (type default))
-  )
   (wire (pts (xy 165.1 86.36) (xy 149.86 86.36))
     (stroke (width 0) (type default))
@@
     (effects (font (size 1.27 1.27)) (justify left bottom))
   )
-  (text "UART2" (at 223.52 57.15 0)
-    (effects (font (size 1.27 1.27)) (justify left bottom))
-  )
   (text "Virtual ground for DUT\ncurrent measurement" (at 86.36 120.65 0)
     (effects (font (size 1.27 1.27)) (justify left bottom))
@@
     (effects (font (size 1.27 1.27)) (justify right bottom))
   )
-  (label "D10_MCU_TX" (at 209.55 57.15 0) (fields_autoplaced)
+  (label "D4_MCU_PC1" (at 151.13 88.9 0) (fields_autoplaced)
     (effects (font (size 1.27 1.27)) (justify left bottom))
   )
@@
     (effects (font (size 1.27 1.27)) (justify left bottom))
   )
+  (label "D4_MCU_PC1" (at 54.61 81.28 270) (fields_autoplaced)
+    (effects (font (size 1.27 1.27)) (justify right bottom))
+  )
   (label "D3_MCU_PC0" (at 163.83 86.36 180) (fields_autoplaced)
     (effects (font (size 1.27 1.27)) (justify right bottom))
@@
     (effects (font (size 1.27 1.27)) (justify left bottom))
   )
-  (label "D9_MCU_RX" (at 210.82 54.61 0) (fields_autoplaced)
-    (effects (font (size 1.27 1.27)) (justify left bottom))
-  )
