File: daughter-board/stm32l462/stm32l462.kicad_pcb (KiCad board)
At the start: 2 copper layers, 33 x 91.4 mm, 49 parts, among them J1 Conn_02x10_Odd_Even, J2 Conn_02x10_Odd_Even, U1 STM32L476RG, Y1 Crystal_Small

Commit message: Change package folder name - Add integration test and actions script
Parts:
- removed C1: 100n, Capacitor_SMD:C_0805_2012Metric
- U1: value STM32L476RG -> STM32L462CETx; footprint mykicadlibs:ALLSOCKET-QFP64 -> Package_QFP:LQFP-48_7x7mm_P0.5mm
- moved U1 1.30 mm to (172.0, 85.0), turned to 0 degrees
Connections:
- J1 pad 3: /D3_MCU_PC0 -> /D3_MCU_PB0
- J1 pad 6: /D4_MCU_PC1 -> /D4_MCU_PB1
- U1 pad 1: unconnected-(U1-VBAT-Pad1) -> +3V3
- U1 pad 12: GNDA -> unconnected-(U1-PA2-Pad12)
- U1 pad 13: +3V3 -> unconnected-(U1-PA3-Pad13)
- U1 pad 18: GNDA -> /D3_MCU_PB0
- U1 pad 19: +3V3 -> /D4_MCU_PB1
- U1 pad 23: unconnected-(U1-PA7-Pad23) -> GNDA
- U1 pad 24: unconnected-(U1-PC4-Pad24) -> +3V3
- U1 pad 28: /D7_BOOT1 -> unconnected-(U1-PB15-Pad28)
- U1 pad 30: unconnected-(U1-PB11-Pad30) -> /D1_MCU_TX
- U1 pad 31: unconnected-(U1-VCAP_1-Pad31) -> /D0_MCU_RX
- U1 pad 32: +3V3 -> unconnected-(U1-PA11-Pad32)
- U1 pad 35: unconnected-(U1-PB14-Pad35) -> GNDA
- U1 pad 36: unconnected-(U1-PB15-Pad36) -> +3V3
- U1 pad 42: /D1_MCU_TX -> unconnected-(U1-PB6-Pad42)
- U1 pad 43: /D0_MCU_RX -> unconnected-(U1-PB7-Pad43)
- U1 pad 44: unconnected-(U1-PA11-Pad44) -> /D6_BOOT0
- U1 pad 47: unconnected-(U1-VCAP_2-Pad47) -> GNDA
- U1 pad 8: /D3_MCU_PC0 -> GNDA
- U1 pad 9: /D4_MCU_PC1 -> +3V3
Routing:
- net +3V3: track 125.9 -> 2.87 mm
- net GNDA: track 81.7 -> 4.81 mm
- net /D4_MCU_PC1: track 51.9 -> 0.00 mm
- net /D0_MCU_RX: track 48.1 -> 0.00 mm
- net /D6_BOOT0: track 48.7 -> 3.59 mm
- net /D2_NRST: track 52.1 -> 8.73 mm
- net /D3_MCU_PC0: track 43.1 -> 0.00 mm
- net /D7_BOOT1: track 41.5 -> 0.00 mm
- net /D1_MCU_TX: track 50.6 -> 34.5 mm
- net Net-(U1-PH0): track 18.6 -> 4.00 mm
- net Net-(U1-PH1): track 19.1 -> 4.80 mm
- net /D4_MCU_PB1: track 0.00 -> 4.62 mm
- net /D3_MCU_PB0: track 0.00 -> 1.66 mm
Other:
- board text added: "D0: MCU RX D1: MCU TX D2: NRST D3: PB0 D4: PB1 D6: BOOT0"
- board text added: "STM32L462CEUx QFP64"
- board text removed: "D0: MCU RX D1: MCU TX D2: NRST D3: PC0 D6: BOOT0 D7: BOOT1"
- board text removed: "STM32L476 QFP64 socket"

Commit message: l462 routing -  Add ATMega board - Update ceval script
Parts:
- added C1: 100n, PCM_Capacitor_SMD_AKL:C_0805_2012Metric, F.Cu at (180.6, 82.9)
- moved U1 1.43 mm to (170.7, 84.5), turned to -90 degrees
Connections:
- J1 pad 7: /D7_BOOT1 -> unconnected-(J1-Pin_7-Pad7)
- U1 pad 2: unconnected-(U1-PC13-Pad2) -> /D3_MCU_PC13
- U1 pad 3: unconnected-(U1-PC14-Pad3) -> /D4_MCU_PC14
Routing:
- net GNDA: track 4.81 -> 106.0 mm, vias 1 -> 4
- net +3V3: track 2.87 -> 89.1 mm, vias 0 -> 5
- net /D6_BOOT0: track 3.59 -> 48.7 mm, vias 0 -> 1
- net /D3_MCU_PB0: track 1.66 -> 45.4 mm, vias 0 -> 1
- net /D0_MCU_RX: track 0.00 -> 42.8 mm
- net /D2_NRST: track 8.73 -> 49.5 mm, vias 0 -> 3
- net /D4_MCU_PB1: track 4.62 -> 40.1 mm, vias 0 -> 1
- net Net-(U1-PH1): track 4.80 -> 26.2 mm, vias 0 -> 1
- net Net-(U1-PH0): track 4.00 -> 21.1 mm, vias 0 -> 1
- net /D1_MCU_TX: track 34.5 -> 47.6 mm
