File: daughter-board/AtMega328p/AtMega328p.kicad_pcb (KiCad board)
At the start: 2 copper layers, 43.2 x 91.7 mm, 51 parts, among them J1 Conn_02x10_Odd_Even, J2 Conn_02x10_Odd_Even, U1 MAX4619CPE_, U2 ATmega328P-P, Y1 Crystal_Small

Commit message: Update atmega board
Parts:
- removed C1: 100n, PCM_Capacitor_SMD_AKL:C_0201_0603Metric
- moved U1 5.71 mm to (185.5, 73.4)
Connections:
- net +3V3 renamed VDDA
- net +5V renamed Net-(J3-Pin_2)
- C3 pad 2: Net-(U2-XTAL1/PB6) -> /D7_CLK_PB6
- J1 pad 7: unconnected-(J1-Pin_7-Pad7) -> /D7_CLK_PB6
- R1 pad 1: Net-(U2-XTAL1/PB6) -> /D7_CLK_PB6
- U2 pad 9: Net-(U2-XTAL1/PB6) -> /D7_CLK_PB6
- Y1 pad 2: Net-(U2-XTAL1/PB6) -> /D7_CLK_PB6
Routing:
- net /D7_CLK_PB6: track 0.00 -> 32.8 mm
- net Net-(U2-XTAL1/PB6): track 7.43 -> 0.00 mm
